File: PCB/zHeat_PCB.kicad_sch (KiCad schematic)
At the start: 86 parts, among them IC1 MAX14932AASE+, IC2 RMB6S, IC3 RMB6S, J1 USB4110GFA, J2 WAGO 250-202, J3 WAGO 250-202, J4 WAGO 250-202, Q1 BC847BS, U1 ESP32-C6-WROOM-1, U2 LM2735X (1.6MHz), U3 MCP1826S-3302E/DB, U4 MAX22088GTG_

Commit message: PCB and Enclosure ready
Parts:
- C11: symbol Device:C -> Device:C_Polarized
Changed lines of the file:
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@@
 	)
 	(symbol
-		(lib_id "Device:C")
+		(lib_id "Device:C_Polarized")
 		(at 248.92 157.48 0)
 		(unit 1)
@@
 			)
 		)
-		(property "Description" "Unpolarized capacitor"
+		(property "Description" "Polarized capacitor"
 			(at 248.92 157.48 0)
 			(hide yes)
